File: keyboard.sch (KiCad schematic (older format))
At the start: 6 parts

Commit message: update micro system
Parts:
- added C? (x2): 22p, symbol keyboard_parts:C
- added C?: 0.1u, symbol keyboard_parts:C
- added C?: 1u, symbol keyboard_parts:C
- added C?: 4.7u, symbol keyboard_parts:C
- added SW?: SW_PUSH, symbol keyboard_parts:SW_PUSH
- added X?: 16Mhz, symbol keyboard_parts:XTAL
Connections:
- net labels added: +5V, PE6, VUSB, VUSB_RAW
- net labels removed: VBUS
- wire segments 23 -> 43
Changed lines of the file:
@@
 Connection ~ 1650 950
 Text GLabel 4800 850  2    50   Input ~ 0
-VBUS
-Wire Wire Line
-	1650 850  4300 850
-Connection ~ 1650 850
-Wire Wire Line
-	5550 2150 4300 2150
+VUSB
 Wire Wire Line
 	4300 2150 4300 1650
-Connection ~ 4300 850
 Wire Wire Line
 	4300 850  4800 850
@@
 	1150 3750 1150 4100
 Connection ~ 1150 3750
+$Comp
+L keyboard_parts:XTAL X?
+U 1 1 5BBC32C3
+P 4450 3450
+F 0 "X?" H 4450 3742 60  0000 C CNN
+F 1 "16Mhz" H 4450 3636 60  0000 C CNN
+F 2 "" H 4450 3450 60  0000 C CNN
+F 3 "" H 4450 3450 60  0000 C CNN
+	1    4450 3450
+	1    0    0    -1
+$EndComp
+Wire Wire Line
+	5550 3050 4150 3050
+Wire Wire Line
+	4150 3050 4150 3450
+Wire Wire Line
+	5550 3150 4750 3150
+Wire Wire Line
+	4750 3150 4750 3450
+$Comp
+L keyboard_parts:C C?
+U 1 1 5BBC4166
+P 4150 3650
+F 0 "C?" H 4280 3696 50  0000 L CNN
+F 1 "22p" H 4280 3605 50  0000 L CNN
+F 2 "" H 4150 3650 60  0000 C CNN
+F 3 "" H 4150 3650 60  0000 C CNN
+	1    4150 3650
+	1    0    0    -1
+$EndComp
+Connection ~ 4150 3450
+$Comp
+L keyboard_parts:C C?
+U 1 1 5BBC41C7
+P 4750 3650
+F 0 "C?" H 4880 3696 50  0000 L CNN
+F 1 "22p" H 4880 3605 50  0000 L CNN
+F 2 "" H 4750 3650 60  0000 C CNN
+F 3 "" H 4750 3650 60  0000 C CNN
+	1    4750 3650
+	1    0    0    -1
+$EndComp
+Connection ~ 4750 3450
+$Comp
+L power:GND #PWR?
+U 1 1 5BBC4228
+P 4750 3850
+F 0 "#PWR?" H 4750 3600 50  0001 C CNN
+F 1 "GND" H 4755 3677 50  0000 C CNN
+F 2 "" H 4750 3850 50  0001 C CNN
+F 3 "" H 4750 3850 50  0001 C CNN
+	1    4750 3850
+	1    0    0    -1
+$EndComp
+$Comp
+L power:GND #PWR?
+U 1 1 5BBC427E
+P 4150 3850
+F 0 "#PWR?" H 4150 3600 50  0001 C CNN
+F 1 "GND" H 4155 3677 50  0000 C CNN
+F 2 "" H 4150 3850 50  0001 C CNN
+F 3 "" H 4150 3850 50  0001 C CNN
+	1    4150 3850
+	1    0    0    -1
+$EndComp
+Text Label 5350 1550 0    50   ~ 0
+PE6
+Wire Wire Line
+	5550 1550 5350 1550
+$Comp
+L keyboard_parts:SW_PUSH SW?
+U 1 1 5BBDE8F3
+P 4400 2750
+F 0 "SW?" H 4400 3005 50  0000 C CNN
+F 1 "SW_PUSH" H 4400 2914 50  0000 C CNN
+F 2 "" H 4400 2750 60  0000 C CNN
+F 3 "" H 4400 2750 60  0000 C CNN
+	1    4400 2750
+	1    0    0    -1
+$EndComp
+Wire Wire Line
+	5550 2750 4700 2750
+$Comp
+L power:GND #PWR?
+U 1 1 5BBDEE37
+P 3900 3850
+F 0 "#PWR?" H 3900 3600 50  0001 C CNN
+F 1 "GND" H 3905 3677 50  0000 C CNN
+F 2 "" H 3900 3850 50  0001 C CNN
+F 3 "" H 3900 3850 50  0001 C CNN
+	1    3900 3850
+	1    0    0    -1
+$EndComp
+Wire Wire Line
+	3900 2750 4100 2750
+Wire Wire Line
+	3900 2750 3900 3850
+$Comp
+L power:GND #PWR?
+U 1 1 5BBDF377
+P 3650 3850
+F 0 "#PWR?" H 3650 3600 50  0001 C CNN
+F 1 "GND" H 3655 3677 50  0000 C CNN
+F 2 "" H 3650 3850 50  0001 C CNN
+F 3 "" H 3650 3850 50  0001 C CNN
+	1    3650 3850
+	1    0    0    -1
+$EndComp
+Wire Wire Line
+	5550 1950 3650 1950
+Wire Wire Line
+	3650 1950 3650 2950
+Wire Wire Line
+	5550 2950 3650 2950
+Connection ~ 3650 2950
+Wire Wire Line
+	3650 2950 3650 3850
+$Comp
+L keyboard_parts:C C?
+U 1 1 5BBDFDF9
+P 3350 3550
+F 0 "C?" H 3480 3596 50  0000 L CNN
+F 1 "0.1u" H 3480 3505 50  0000 L CNN
+F 2 "" H 3350 3550 60  0000 C CNN
+F 3 "" H 3350 3550 60  0000 C CNN
+	1    3350 3550
+	1    0    0    -1
+$EndComp
+$Comp
+L keyboard_parts:C C?
+U 1 1 5BBDFE63
+P 3900 2250
+F 0 "C?" H 4030 2296 50  0000 L CNN
+F 1 "1u" H 4030 2205 50  0000 L CNN
+F 2 "" H 3900 2250 60  0000 C CNN
+F 3 "" H 3900 2250 60  0000 C CNN
+	1    3900 2250
+	1    0    0    -1
+$EndComp
+Wire Wire Line
+	5550 2050 3900 2050
+$Comp
+L power:GND #PWR?
+U 1 1 5BBE044A
+P 3900 2500
+F 0 "#PWR?" H 3900 2250 50  0001 C CNN
+F 1 "GND" H 3905 2327 50  0000 C CNN
+F 2 "" H 3900 2500 50  0001 C CNN
+F 3 "" H 3900 2500 50  0001 C CNN
+	1    3900 2500
+	1    0    0    -1
+$EndComp
+$Comp
+L power:GND #PWR?
+U 1 1 5BBE0497
+P 3350 3850
+F 0 "#PWR?" H 3350 3600 50  0001 C CNN
+F 1 "GND" H 3355 3677 50  0000 C CNN
+F 2 "" H 3350 3850 50  0001 C CNN
+F 3 "" H 3350 3850 50  0001 C CNN
+	1    3350 3850
+	1    0    0    -1
+$EndComp
+Wire Wire Line
+	3350 3750 3350 3850
+Wire Wire Line
+	3900 2450 3900 2500
+$Comp
+L keyboard_parts:+5V #PWR?
+U 1 1 5BBE1511
+P 3350 2400
+F 0 "#PWR?" H 3350 2370 20  0001 C CNN
+F 1 "+5V" H 3350 2538 30  0000 C CNN
+F 2 "" H 3350 2400 60  0000 C CNN
+F 3 "" H 3350 2400 60  0000 C CNN
+	1    3350 2400
+	1    0    0    -1
+$EndComp
+Wire Wire Line
+	3350 2400 3350 2850
+Wire Wire Line
+	5550 2850 3350 2850
+Connection ~ 3350 2850
+Wire Wire Line
+	3350 2850 3350 3350
+Text Label 5300 2150 0    50   ~ 0
+VUSB
+Wire Wire Line
+	4300 2150 5550 2150
+Text Label 2150 850  2    50   ~ 0
+VUSB_RAW
+Text Label 3650 850  0    50   ~ 0
+VUSB
+Wire Wire Line
+	1650 850  4300 850
+Connection ~ 1650 850
+Connection ~ 4300 850
+$Comp
+L keyboard_parts:C C?
+U 1 1 5BBE37E5
+P 3000 3550
+F 0 "C?" H 3130 3596 50  0000 L CNN
+F 1 "4.7u" H 3130 3505 50  0000 L CNN
+F 2 "" H 3000 3550 60  0000 C CNN
+F 3 "" H 3000 3550 60  0000 C CNN
+	1    3000 3550
+	1    0    0    -1
+$EndComp
+$Comp
+L power:GND #PWR?
+U 1 1 5BBE3899
+P 3000 3850
+F 0 "#PWR?" H 3000 3600 50  0001 C CNN
+F 1 "GND" H 3005 3677 50  0000 C CNN
+F 2 "" H 3000 3850 50  0001 C CNN
+F 3 "" H 3000 3850 50  0001 C CNN
+	1    3000 3850
+	1    0    0    -1
+$EndComp
+$Comp
+L keyboard_parts:+5V #PWR?
+U 1 1 5BBE38F0
+P 3000 2400
+F 0 "#PWR?" H 3000 2370 20  0001 C CNN
+F 1 "+5V" H 3000 2538 30  0000 C CNN
+F 2 "" H 3000 2400 60  0000 C CNN
+F 3 "" H 3000 2400 60  0000 C CNN
+	1    3000 2400
+	1    0    0    -1
+$EndComp
+Wire Wire Line
+	3000 2400 3000 3350
+Wire Wire Line
+	3000 3750 3000 3850
 $EndSCHEMATC

Commit message: matrix layout
Parts:
- added C6, C7, C8: 0.1u, symbol keyboard_parts:C
- added R5: 1k, symbol keyboard_parts:R
- gave numbers to parts that had none: 13
Connections:
- net labels added: PB0, PB1, PB3, PB7, ~RESET
- wire segments 43 -> 71

Commit message: layout
Connections:
- net labels added: COL0, COL1, COL2, COL3, COL4, PB2, PB4, PB5, PB6, PC6, PC7, ROW0, ROW1, ROW2, ROW3, ROW4
- wire segments 71 -> 86
Changed lines of the file:
@@
 F 0 "U1" H 6625 3937 60  0000 C CNN
 F 1 "ATMEGA32U4" H 6625 3831 60  0000 C CNN
-F 2 "keyboard_parts:QFP44" H 6600 2600 60  0000 C CNN
+F 2 "keyboard_parts:QFP44" H 6600 2600 60  0001 C CNN
 F 3 "" H 6600 2600 60  0000 C CNN
 	1    6600 2600
@@
 PB1
 Text Label 5400 2450 0    50   ~ 0
-PB3
+PB2
 Text Label 5400 2550 0    50   ~ 0
 PB3
@@
 F1 "key.sch" 50
 $EndSheet
+Text Label 7850 3150 2    50   ~ 0
+PB4
+Text Label 7850 3050 2    50   ~ 0
+PB5
+Text Label 7850 2950 2    50   ~ 0
+PB6
+Wire Wire Line
+	7700 2950 7850 2950
+Wire Wire Line
+	7700 3050 7850 3050
+Wire Wire Line
+	7700 3150 7850 3150
+Text Label 6150 4750 0    50   ~ 0
+PB0
+Text Label 6150 4900 0    50   ~ 0
+PB1
+Text Label 6150 5050 0    50   ~ 0
+PB2
+Text Label 6150 5200 0    50   ~ 0
+PB3
+Text Label 6150 5350 0    50   ~ 0
+PB4
+Text Label 6150 5500 0    50   ~ 0
+PB5
+Text Label 6150 5650 0    50   ~ 0
+PB6
+Text Label 6150 5800 0    50   ~ 0
+PB7
+Text GLabel 6700 4750 2    50   Input ~ 0
+ROW0
+Text GLabel 6700 4900 2    50   Input ~ 0
+ROW1
+Text GLabel 6700 5050 2    50   Input ~ 0
+ROW2
+Text GLabel 6700 5200 2    50   Input ~ 0
+ROW3
+Text GLabel 6700 5350 2    50   Input ~ 0
+ROW4
+Text GLabel 6700 5500 2    50   Input ~ 0
+COL0
+Text GLabel 6700 5650 2    50   Input ~ 0
+COL1
+Text GLabel 6700 5800 2    50   Input ~ 0
+COL2
+Wire Wire Line
+	6150 4750 6700 4750
+Wire Wire Line
+	6150 4900 6700 4900
+Wire Wire Line
+	6150 5050 6700 5050
+Wire Wire Line
+	6150 5200 6700 5200
+Wire Wire Line
+	6150 5350 6700 5350
+Wire Wire Line
+	6150 5500 6700 5500
+Wire Wire Line
+	6150 5650 6700 5650
+Wire Wire Line
+	6150 5800 6700 5800
+Text Label 7850 2850 2    50   ~ 0
+PC6
+Text Label 7850 2750 2    50   ~ 0
+PC7
+Wire Wire Line
+	7700 2750 7850 2750
+Wire Wire Line
+	7700 2850 7850 2850
+Text Label 6150 5950 0    50   ~ 0
+PC6
+Text Label 6150 6100 0    50   ~ 0
+PC7
+Text GLabel 6700 5950 2    50   Input ~ 0
+COL3
+Text GLabel 6700 6100 2    50   Input ~ 0
+COL4
+Wire Wire Line
+	6700 5950 6150 5950
+Wire Wire Line
+	6150 6100 6700 6100
 $EndSCHEMATC
