File: key.sch (KiCad schematic (older format))
At the start: 122 parts

Commit message: matrix layout
Parts:
- removed D1, D10, D11, D12, D13, D14, D15, D16, D17, D18, D19, D2, D20, D21, D22, D23, D24, D25, D26, D27, D28, D29, D3, D30, D31, D32, D33, D34, D35, D36, D37, D38, D39, D4, D40, D41, D42, D43, D44, D45, D46, D47, D48, D49, D5, D50, D51, D52, D53, D54, D55, D56, D57, D58, D59, D6, D60, D61, D7, D8, D9: 1N4148, 0805:0805D, symbol DIODE
- removed S1, S10, S11, S12, S13, S14, S15, S16, S17, S18, S19, S2, S20, S21, S22, S23, S24, S25, S26, S27, S28, S29, S3, S30, S31, S32, S33, S34, S35, S36, S37, S38, S39, S4, S40, S41, S42, S43, S44, S45, S46, S47, S48, S49, S5, S50, S51, S52, S53, S54, S55, S56, S57, S58, S59, S6, S60, S61, S7, S8, S9: MX1A, mx1a:MX1A, symbol MX1A
- added D1, D10, D11, D12, D13, D14, D15, D16, D17, D18, D19, D2, D20, D21, D22, D23, D24, D25, D26, D27, D28, D29, D3, D30, D31, D32, D33, D34, D35, D36, D37, D38, D39, D4, D40, D41, D42, D43, D44, D45, D46, D47, D48, D49, D5, D50, D51, D52, D53, D54, D55, D56, D57, D58, D59, D6, D60, D61, D62, D63, D64, D7, D8, D9: D, symbol keyboard_parts:D
- added SW10: 8, Button_Switch_Keyboard:SW_Cherry_MX1A_1.00u_PCB, symbol keyboard_parts:SW_PUSH
- added SW11: 9, Button_Switch_Keyboard:SW_Cherry_MX1A_1.00u_PCB, symbol keyboard_parts:SW_PUSH
- added SW12: 0, Button_Switch_Keyboard:SW_Cherry_MX1A_1.00u_PCB, symbol keyboard_parts:SW_PUSH
- added SW13: -, Button_Switch_Keyboard:SW_Cherry_MX1A_1.00u_PCB, symbol keyboard_parts:SW_PUSH
- added SW14: =, Button_Switch_Keyboard:SW_Cherry_MX1A_1.00u_PCB, symbol keyboard_parts:SW_PUSH
- added SW15: delete, Button_Switch_Keyboard:SW_Cherry_MX1A_2.00u_PCB, symbol keyboard_parts:SW_PUSH
- added SW16: tab, Button_Switch_Keyboard:SW_Cherry_MX1A_1.50u_PCB, symbol keyboard_parts:SW_PUSH
- added SW17: q, Button_Switch_Keyboard:SW_Cherry_MX1A_1.00u_PCB, symbol keyboard_parts:SW_PUSH
- added SW18: w, Button_Switch_Keyboard:SW_Cherry_MX1A_1.00u_PCB, symbol keyboard_parts:SW_PUSH
- added SW19: e, Button_Switch_Keyboard:SW_Cherry_MX1A_1.00u_PCB, symbol keyboard_parts:SW_PUSH
- added SW2: ESC, Button_Switch_Keyboard:SW_Cherry_MX1A_1.00u_PCB, symbol keyboard_parts:SW_PUSH
- added SW20: r, Button_Switch_Keyboard:SW_Cherry_MX1A_1.00u_PCB, symbol keyboard_parts:SW_PUSH
- added SW21: t, Button_Switch_Keyboard:SW_Cherry_MX1A_1.00u_PCB, symbol keyboard_parts:SW_PUSH
- added SW22: y, Button_Switch_Keyboard:SW_Cherry_MX1A_1.00u_PCB, symbol keyboard_parts:SW_PUSH
- added SW23: u, Button_Switch_Keyboard:SW_Cherry_MX1A_1.00u_PCB, symbol keyboard_parts:SW_PUSH
- added SW24: i, Button_Switch_Keyboard:SW_Cherry_MX1A_1.00u_PCB, symbol keyboard_parts:SW_PUSH
- added SW25: o, Button_Switch_Keyboard:SW_Cherry_MX1A_1.00u_PCB, symbol keyboard_parts:SW_PUSH
- added SW26: p, Button_Switch_Keyboard:SW_Cherry_MX1A_1.00u_PCB, symbol keyboard_parts:SW_PUSH
- added SW27: [, Button_Switch_Keyboard:SW_Cherry_MX1A_1.00u_PCB, symbol keyboard_parts:SW_PUSH
- added SW28: ], Button_Switch_Keyboard:SW_Cherry_MX1A_1.00u_PCB, symbol keyboard_parts:SW_PUSH
- added SW29: \\, Button_Switch_Keyboard:SW_Cherry_MX1A_1.50u_PCB, symbol keyboard_parts:SW_PUSH
- added SW3: 1, Button_Switch_Keyboard:SW_Cherry_MX1A_1.00u_PCB, symbol keyboard_parts:SW_PUSH
- added SW30: lock, Button_Switch_Keyboard:SW_Cherry_MX1A_1.75u_PCB, symbol keyboard_parts:SW_PUSH
- added SW31: a, Button_Switch_Keyboard:SW_Cherry_MX1A_1.00u_PCB, symbol keyboard_parts:SW_PUSH
- added SW32: s, Button_Switch_Keyboard:SW_Cherry_MX1A_1.00u_PCB, symbol keyboard_parts:SW_PUSH
- added SW33: d, Button_Switch_Keyboard:SW_Cherry_MX1A_1.00u_PCB, symbol keyboard_parts:SW_PUSH
- added SW34: f, Button_Switch_Keyboard:SW_Cherry_MX1A_1.00u_PCB, symbol keyboard_parts:SW_PUSH
- added SW35: g, Button_Switch_Keyboard:SW_Cherry_MX1A_1.00u_PCB, symbol keyboard_parts:SW_PUSH
- added SW36: h, Button_Switch_Keyboard:SW_Cherry_MX1A_1.00u_PCB, symbol keyboard_parts:SW_PUSH
- added SW37: j, Button_Switch_Keyboard:SW_Cherry_MX1A_1.00u_PCB, symbol keyboard_parts:SW_PUSH
- added SW38: k, Button_Switch_Keyboard:SW_Cherry_MX1A_1.00u_PCB, symbol keyboard_parts:SW_PUSH
- added SW39: l, Button_Switch_Keyboard:SW_Cherry_MX1A_1.00u_PCB, symbol keyboard_parts:SW_PUSH
- added SW4: 2, Button_Switch_Keyboard:SW_Cherry_MX1A_1.00u_PCB, symbol keyboard_parts:SW_PUSH
- added SW40: ;, Button_Switch_Keyboard:SW_Cherry_MX1A_1.00u_PCB, symbol keyboard_parts:SW_PUSH
- added SW41: ', Button_Switch_Keyboard:SW_Cherry_MX1A_1.00u_PCB, symbol keyboard_parts:SW_PUSH
- added SW42: return, Button_Switch_Keyboard:SW_Cherry_MX1A_2.25u_PCB, symbol keyboard_parts:SW_PUSH
- added SW43: shift, Button_Switch_Keyboard:SW_Cherry_MX1A_2.00u_PCB, symbol keyboard_parts:SW_PUSH
- added SW44: z, Button_Switch_Keyboard:SW_Cherry_MX1A_1.00u_PCB, symbol keyboard_parts:SW_PUSH
- added SW45: x, Button_Switch_Keyboard:SW_Cherry_MX1A_1.00u_PCB, symbol keyboard_parts:SW_PUSH
- added SW46: c, Button_Switch_Keyboard:SW_Cherry_MX1A_1.00u_PCB, symbol keyboard_parts:SW_PUSH
- added SW47: v, Button_Switch_Keyboard:SW_Cherry_MX1A_1.00u_PCB, symbol keyboard_parts:SW_PUSH
- added SW48: b, Button_Switch_Keyboard:SW_Cherry_MX1A_1.00u_PCB, symbol keyboard_parts:SW_PUSH
- added SW49: n, Button_Switch_Keyboard:SW_Cherry_MX1A_1.00u_PCB, symbol keyboard_parts:SW_PUSH
- added SW5: 3, Button_Switch_Keyboard:SW_Cherry_MX1A_1.00u_PCB, symbol keyboard_parts:SW_PUSH
- added SW50: m, Button_Switch_Keyboard:SW_Cherry_MX1A_1.00u_PCB, symbol keyboard_parts:SW_PUSH
- added SW51: ,, Button_Switch_Keyboard:SW_Cherry_MX1A_1.00u_PCB, symbol keyboard_parts:SW_PUSH
- added SW52: ., Button_Switch_Keyboard:SW_Cherry_MX1A_1.00u_PCB, symbol keyboard_parts:SW_PUSH
- added SW53: /, Button_Switch_Keyboard:SW_Cherry_MX1A_1.00u_PCB, symbol keyboard_parts:SW_PUSH
- added SW54: shift, Button_Switch_Keyboard:SW_Cherry_MX1A_1.00u_PCB, symbol keyboard_parts:SW_PUSH
- added SW55: up, Button_Switch_Keyboard:SW_Cherry_MX1A_1.00u_PCB, symbol keyboard_parts:SW_PUSH
- added SW56: delete, Button_Switch_Keyboard:SW_Cherry_MX1A_1.00u_PCB, symbol keyboard_parts:SW_PUSH
- added SW57: fn, Button_Switch_Keyboard:SW_Cherry_MX1A_1.00u_PCB, symbol keyboard_parts:SW_PUSH
- added SW58: control, Button_Switch_Keyboard:SW_Cherry_MX1A_1.25u_PCB, symbol keyboard_parts:SW_PUSH
- added SW59: option, Button_Switch_Keyboard:SW_Cherry_MX1A_1.50u_PCB, symbol keyboard_parts:SW_PUSH
- added SW6: 4, Button_Switch_Keyboard:SW_Cherry_MX1A_1.00u_PCB, symbol keyboard_parts:SW_PUSH
- added SW60, SW62: command, Button_Switch_Keyboard:SW_Cherry_MX1A_1.25u_PCB, symbol keyboard_parts:SW_PUSH
- added SW61: space, Button_Switch_Keyboard:SW_Cherry_MX1A_6.25u_PCB, symbol keyboard_parts:SW_PUSH
- added SW63: left, Button_Switch_Keyboard:SW_Cherry_MX1A_1.00u_PCB, symbol keyboard_parts:SW_PUSH
- added SW64: down, Button_Switch_Keyboard:SW_Cherry_MX1A_1.00u_PCB, symbol keyboard_parts:SW_PUSH
- added SW65: right, Button_Switch_Keyboard:SW_Cherry_MX1A_1.00u_PCB, symbol keyboard_parts:SW_PUSH
- added SW7: 5, Button_Switch_Keyboard:SW_Cherry_MX1A_1.00u_PCB, symbol keyboard_parts:SW_PUSH
- added SW8: 6, Button_Switch_Keyboard:SW_Cherry_MX1A_1.00u_PCB, symbol keyboard_parts:SW_PUSH
- added SW9: 7, Button_Switch_Keyboard:SW_Cherry_MX1A_1.00u_PCB, symbol keyboard_parts:SW_PUSH
Connections:
- net labels added: col1, col10, col11, col12, col13, col14, col2, col3, col4, col5, col6, col7, col8, col9, row1, row2, row3, row4, row5
- wire segments 202 -> 381

Commit message: layout
Connections:
- net labels added: ROW0, ROW1, ROW2, ROW3, ROW4
- net labels removed: row1, row2, row3, row4, row5
- wire segments 381 -> 385
Changed lines of the file:
@@
 Wire Wire Line
 	750  1050 750  1400
-Text HLabel 700  1050 0    50   3State ~ 0
-row1
 Wire Wire Line
 	750  1050 700  1050
@@
 Wire Wire Line
 	1500 2000 1500 2350
-Text HLabel 700  2000 0    50   3State ~ 0
-row2
-Text HLabel 700  2950 0    50   3State ~ 0
-row3
 Wire Wire Line
 	750  3300 750  2950
@@
 Wire Wire Line
 	1500 4850 1500 5200
-Text HLabel 700  3900 0    50   3State ~ 0
-row4
-Text HLabel 700  4850 0    50   3State ~ 0
-row5
 Wire Wire Line
 	1500 2000 2250 2000
@@
 Wire Wire Line
 	9650 5200 9650 5450
+Text GLabel 700  4850 0    50   Input ~ 0
+ROW4
+Text GLabel 700  3900 0    50   Input ~ 0
+ROW3
+Text GLabel 700  2950 0    50   Input ~ 0
+ROW2
+Text GLabel 700  2000 0    50   Input ~ 0
+ROW1
+Text GLabel 700  1050 0    50   Input ~ 0
+ROW0
+Wire Wire Line
+	750  2000 700  2000
+Connection ~ 750  2000
+Wire Wire Line
+	750  2950 700  2950
+Connection ~ 750  2950
+Wire Wire Line
+	750  3900 700  3900
+Connection ~ 750  3900
+Wire Wire Line
+	750  4850 700  4850
+Connection ~ 750  4850
 $EndSCHEMATC

Commit message: pcb layout
Parts:
- D1, D10, D11, D12, D13, D14, D15, D16, D17, D18, D19, D2, D20, D21, D22, D23, D24, D25, D26, D27, D28, D29, D3, D30, D31, D32, D33, D34, D35, D36, D37, D38, D39, D4, D40, D41, D42, D43, D44, D45, D46, D47, D48, D49, D5, D50, D51, D52, D53, D54, D55, D56, D57, D58, D59, D6, D60, D61, D62, D63, D64, D7, D8, D9: footprint (none) -> Diode_SMD:D_0805_2012Metric

Commit message: layout
Parts:
- D1, D10, D11, D12, D13, D14, D15, D16, D17, D18, D19, D2, D20, D21, D22, D23, D24, D25, D26, D27, D28, D29, D3, D30, D31, D32, D33, D34, D35, D36, D37, D38, D39, D4, D40, D41, D42, D43, D44, D45, D46, D47, D48, D49, D5, D50, D51, D52, D53, D54, D55, D56, D57, D58, D59, D6, D60, D61, D62, D63, D64, D7, D8, D9: footprint Diode_SMD:D_0805_2012Metric -> Diode_SMD:D_MiniMELF

Commit message: pcb
Parts:
- SW43: footprint Button_Switch_Keyboard:SW_Cherry_MX1A_2.00u_PCB -> Button_Switch_Keyboard:SW_Cherry_MX1A_2.25u_PCB
- SW54: footprint Button_Switch_Keyboard:SW_Cherry_MX1A_1.00u_PCB -> Button_Switch_Keyboard:SW_Cherry_MX1A_1.75u_PCB
- SW59: footprint Button_Switch_Keyboard:SW_Cherry_MX1A_1.50u_PCB -> Button_Switch_Keyboard:SW_Cherry_MX1A_1.25u_PCB
- SW62: footprint Button_Switch_Keyboard:SW_Cherry_MX1A_1.25u_PCB -> Button_Switch_Keyboard:SW_Cherry_MX1A_1.00u_PCB
Changed lines of the file:
@@
 F 0 "SW43" H 1050 4505 50  0000 C CNN
 F 1 "shift" H 1050 4414 50  0000 C CNN
-F 2 "Button_Switch_Keyboard:SW_Cherry_MX1A_2.00u_PCB" H 1050 4250 60  0001 C CNN
+F 2 "Button_Switch_Keyboard:SW_Cherry_MX1A_2.25u_PCB" H 1050 4250 60  0001 C CNN
 F 3 "" H 1050 4250 60  0000 C CNN
 	1    1050 4250
@@
 F 0 "SW54" H 9350 4505 50  0000 C CNN
 F 1 "shift" H 9350 4414 50  0000 C CNN
-F 2 "Button_Switch_Keyboard:SW_Cherry_MX1A_1.00u_PCB" H 9350 4250 60  0001 C CNN
+F 2 "Button_Switch_Keyboard:SW_Cherry_MX1A_1.75u_PCB" H 9350 4250 60  0001 C CNN
 F 3 "" H 9350 4250 60  0000 C CNN
 	1    9350 4250
@@
 F 0 "SW59" H 2550 5455 50  0000 C CNN
 F 1 "option" H 2550 5364 50  0000 C CNN
-F 2 "Button_Switch_Keyboard:SW_Cherry_MX1A_1.50u_PCB" H 2550 5200 60  0001 C CNN
+F 2 "Button_Switch_Keyboard:SW_Cherry_MX1A_1.25u_PCB" H 2550 5200 60  0001 C CNN
 F 3 "" H 2550 5200 60  0000 C CNN
 	1    2550 5200
@@
 F 0 "SW62" H 4850 5455 50  0000 C CNN
 F 1 "command" H 4850 5364 50  0000 C CNN
-F 2 "Button_Switch_Keyboard:SW_Cherry_MX1A_1.25u_PCB" H 4850 5200 60  0001 C CNN
+F 2 "Button_Switch_Keyboard:SW_Cherry_MX1A_1.00u_PCB" H 4850 5200 60  0001 C CNN
 F 3 "" H 4850 5200 60  0000 C CNN
 	1    4850 5200
