File: keyboard.kicad_pcb (KiCad board)
At the start: 2 copper layers, 70 parts, among them J1 USB_C_Receptacle, SW10 8, SW11 9, SW12 0, SW13 -, SW14 =, SW15 delete, SW16 tab, SW17 q, SW18 w, SW19 e, SW2 ESC, SW20 r, SW21 t, SW22 y, SW23 u, SW24 i, SW25 o, SW26 p, SW27 [, SW28 ], SW29 \, SW3 1, SW30 lock, SW31 a, SW32 s, SW33 d, SW34 f, SW35 g, SW36 h, SW37 j, SW38 k, SW39 l, SW4 2, SW40 ;, SW41 ', SW42 return, SW43 shift, SW44 z, SW45 x, SW46 c, SW47 v, SW48 b, SW49 n, SW5 3, SW50 m, SW51 ,, SW52 ., SW53 /, SW54 shift, SW55 up, SW56 delete, SW57 fn, SW58 control, SW59 option, SW6 4, SW60 command, SW61 space, SW62 command, SW63 left, SW64 down, SW65 right, SW7 5, SW8 6, SW9 7, U1 ATMEGA32U4

Commit message: pcb layout
Parts:
- added D1: D, Diode_SMD:D_0805_2012Metric, B.Cu at (12.7, 46.5)
- added D10: D, Diode_SMD:D_0805_2012Metric, B.Cu at (54.1, 11.4)
- added D11: D, Diode_SMD:D_0805_2012Metric, B.Cu at (64.5, 19.6)
- added D12: D, Diode_SMD:D_0805_2012Metric, B.Cu at (54.1, 9.41)
- added D13: D, Diode_SMD:D_0805_2012Metric, B.Cu at (57.6, 13.5)
- added D14: D, Diode_SMD:D_0805_2012Metric, B.Cu at (61.0, 15.5)
- added D15: D, Diode_SMD:D_0805_2012Metric, B.Cu at (64.5, 17.6)
- added D16: D, Diode_SMD:D_0805_2012Metric, B.Cu at (57.6, 11.4)
- added D17: D, Diode_SMD:D_0805_2012Metric, B.Cu at (54.1, 7.37)
- added D18: D, Diode_SMD:D_0805_2012Metric, B.Cu at (67.9, 19.6)
- added D19: D, Diode_SMD:D_0805_2012Metric, B.Cu at (57.6, 9.41)
- added D2: D, Diode_SMD:D_0805_2012Metric, B.Cu at (54.1, 17.6)
- added D20: D, Diode_SMD:D_0805_2012Metric, B.Cu at (61.0, 13.5)
- added D21: D, Diode_SMD:D_0805_2012Metric, B.Cu at (64.5, 15.5)
- added D22: D, Diode_SMD:D_0805_2012Metric, B.Cu at (46.1, 7.11)
- added D23: D, Diode_SMD:D_0805_2012Metric, B.Cu at (67.9, 17.6)
- added D24: D, Diode_SMD:D_0805_2012Metric, B.Cu at (61.0, 11.4)
- added D25: D, Diode_SMD:D_0805_2012Metric, B.Cu at (57.6, 7.37)
- added D26: D, Diode_SMD:D_0805_2012Metric, B.Cu at (71.4, 19.6)
- added D27: D, Diode_SMD:D_0805_2012Metric, B.Cu at (61.0, 9.41)
- added D28: D, Diode_SMD:D_0805_2012Metric, B.Cu at (64.5, 13.5)
- added D29: D, Diode_SMD:D_0805_2012Metric, B.Cu at (67.9, 15.5)
- added D3: D, Diode_SMD:D_0805_2012Metric, B.Cu at (57.6, 19.6)
- added D30: D, Diode_SMD:D_0805_2012Metric, B.Cu at (57.6, 5.33)
- added D31: D, Diode_SMD:D_0805_2012Metric, B.Cu at (71.4, 17.6)
- added D32: D, Diode_SMD:D_0805_2012Metric, B.Cu at (64.5, 11.4)
- added D33: D, Diode_SMD:D_0805_2012Metric, B.Cu at (61.0, 7.37)
- added D34: D, Diode_SMD:D_0805_2012Metric, B.Cu at (74.8, 19.6)
- added D35: D, Diode_SMD:D_0805_2012Metric, B.Cu at (64.5, 9.41)
- added D36: D, Diode_SMD:D_0805_2012Metric, B.Cu at (67.9, 13.5)
- added D37: D, Diode_SMD:D_0805_2012Metric, B.Cu at (71.4, 15.5)
- added D38: D, Diode_SMD:D_0805_2012Metric, B.Cu at (61.0, 5.33)
- added D39: D, Diode_SMD:D_0805_2012Metric, B.Cu at (74.8, 17.6)
- added D4: D, Diode_SMD:D_0805_2012Metric, B.Cu at (54.1, 15.5)
- added D40: D, Diode_SMD:D_0805_2012Metric, B.Cu at (67.9, 11.4)
- added D41: D, Diode_SMD:D_0805_2012Metric, B.Cu at (64.5, 7.37)
- added D42: D, Diode_SMD:D_0805_2012Metric, B.Cu at (78.3, 19.6)
- added D43: D, Diode_SMD:D_0805_2012Metric, B.Cu at (67.9, 9.41)
- added D44: D, Diode_SMD:D_0805_2012Metric, B.Cu at (71.4, 13.5)
- added D45: D, Diode_SMD:D_0805_2012Metric, B.Cu at (74.8, 15.5)
- added D46: D, Diode_SMD:D_0805_2012Metric, B.Cu at (64.5, 5.33)
- added D47: D, Diode_SMD:D_0805_2012Metric, B.Cu at (78.3, 17.6)
- added D48: D, Diode_SMD:D_0805_2012Metric, B.Cu at (71.4, 11.4)
- added D49: D, Diode_SMD:D_0805_2012Metric, B.Cu at (67.9, 7.37)
- added D5: D, Diode_SMD:D_0805_2012Metric, B.Cu at (57.6, 17.6)
- added D50: D, Diode_SMD:D_0805_2012Metric, B.Cu at (81.7, 19.6)
- added D51: D, Diode_SMD:D_0805_2012Metric, B.Cu at (71.4, 9.41)
- added D52: D, Diode_SMD:D_0805_2012Metric, B.Cu at (74.8, 13.5)
- added D53: D, Diode_SMD:D_0805_2012Metric, B.Cu at (78.3, 15.5)
- added D54: D, Diode_SMD:D_0805_2012Metric, B.Cu at (67.9, 5.33)
- added D55: D, Diode_SMD:D_0805_2012Metric, B.Cu at (81.7, 17.6)
- added D56: D, Diode_SMD:D_0805_2012Metric, B.Cu at (74.8, 11.4)
- added D57: D, Diode_SMD:D_0805_2012Metric, B.Cu at (71.4, 7.37)
- added D58: D, Diode_SMD:D_0805_2012Metric, B.Cu at (74.8, 9.41)
- added D59: D, Diode_SMD:D_0805_2012Metric, B.Cu at (78.3, 13.5)
- added D6: D, Diode_SMD:D_0805_2012Metric, B.Cu at (61.0, 19.6)
- added D60: D, Diode_SMD:D_0805_2012Metric, B.Cu at (81.7, 15.5)
- added D61: D, Diode_SMD:D_0805_2012Metric, B.Cu at (71.4, 5.33)
- added D62: D, Diode_SMD:D_0805_2012Metric, B.Cu at (78.3, 11.4)
- added D63: D, Diode_SMD:D_0805_2012Metric, B.Cu at (74.8, 7.37)
- added D64: D, Diode_SMD:D_0805_2012Metric, B.Cu at (78.3, 9.41)
- added D7: D, Diode_SMD:D_0805_2012Metric, B.Cu at (54.1, 13.5)
- added D8: D, Diode_SMD:D_0805_2012Metric, B.Cu at (57.6, 15.5)
- added D9: D, Diode_SMD:D_0805_2012Metric, B.Cu at (61.0, 17.6)
Connections:
- net /PB7 renamed COL2
- net Net-(U1-Pad29) renamed COL0
- net Net-(U1-Pad30) renamed COL1
- net Net-(U1-Pad31) renamed COL3
- net Net-(U1-Pad32) renamed COL4
- SW10 pad 1: /key/row1 -> ROW0
- SW11 pad 1: /key/row1 -> ROW0
- SW12 pad 1: /key/row1 -> ROW0
- SW13 pad 1: /key/row1 -> ROW0
- SW14 pad 1: /key/row1 -> ROW0
- SW15 pad 1: /key/row1 -> ROW0
- SW16 pad 1: Net-(SW16-Pad1) -> ROW1
- SW17 pad 1: Net-(SW16-Pad1) -> ROW1
- SW18 pad 1: Net-(SW16-Pad1) -> ROW1
- SW19 pad 1: Net-(SW16-Pad1) -> ROW1
- SW2 pad 1: /key/row1 -> ROW0
- SW20 pad 1: Net-(SW16-Pad1) -> ROW1
- SW21 pad 1: Net-(SW16-Pad1) -> ROW1
- SW22 pad 1: Net-(SW16-Pad1) -> ROW1
- SW23 pad 1: Net-(SW16-Pad1) -> ROW1
- SW24 pad 1: Net-(SW16-Pad1) -> ROW1
- SW25 pad 1: Net-(SW16-Pad1) -> ROW1
- SW26 pad 1: Net-(SW16-Pad1) -> ROW1
- SW27 pad 1: Net-(SW16-Pad1) -> ROW1
- SW28 pad 1: Net-(SW16-Pad1) -> ROW1
- SW29 pad 1: Net-(SW16-Pad1) -> ROW1
- SW3 pad 1: /key/row1 -> ROW0
- SW30 pad 1: Net-(SW30-Pad1) -> ROW2
- SW31 pad 1: Net-(SW30-Pad1) -> ROW2
- SW32 pad 1: Net-(SW30-Pad1) -> ROW2
- SW33 pad 1: Net-(SW30-Pad1) -> ROW2
- SW34 pad 1: Net-(SW30-Pad1) -> ROW2
- SW35 pad 1: Net-(SW30-Pad1) -> ROW2
- SW36 pad 1: Net-(SW30-Pad1) -> ROW2
- SW37 pad 1: Net-(SW30-Pad1) -> ROW2
- SW38 pad 1: Net-(SW30-Pad1) -> ROW2
- SW39 pad 1: Net-(SW30-Pad1) -> ROW2
- SW4 pad 1: /key/row1 -> ROW0
- SW40 pad 1: Net-(SW30-Pad1) -> ROW2
- SW41 pad 1: Net-(SW30-Pad1) -> ROW2
- SW42 pad 1: Net-(SW30-Pad1) -> ROW2
- SW43 pad 1: Net-(SW43-Pad1) -> ROW3
- SW44 pad 1: Net-(SW43-Pad1) -> ROW3
- SW45 pad 1: Net-(SW43-Pad1) -> ROW3
- SW46 pad 1: Net-(SW43-Pad1) -> ROW3
- SW47 pad 1: Net-(SW43-Pad1) -> ROW3
- SW48 pad 1: Net-(SW43-Pad1) -> ROW3
- SW49 pad 1: Net-(SW43-Pad1) -> ROW3
- SW5 pad 1: /key/row1 -> ROW0
- SW50 pad 1: Net-(SW43-Pad1) -> ROW3
- SW51 pad 1: Net-(SW43-Pad1) -> ROW3
- SW52 pad 1: Net-(SW43-Pad1) -> ROW3
- SW53 pad 1: Net-(SW43-Pad1) -> ROW3
- SW54 pad 1: Net-(SW43-Pad1) -> ROW3
- SW55 pad 1: Net-(SW43-Pad1) -> ROW3
- SW56 pad 1: Net-(SW43-Pad1) -> ROW3
- SW57 pad 1: Net-(SW57-Pad1) -> ROW4
- SW58 pad 1: Net-(SW57-Pad1) -> ROW4
- SW59 pad 1: Net-(SW57-Pad1) -> ROW4
- SW6 pad 1: /key/row1 -> ROW0
- SW60 pad 1: Net-(SW57-Pad1) -> ROW4
- SW61 pad 1: Net-(SW57-Pad1) -> ROW4
- SW62 pad 1: Net-(SW57-Pad1) -> ROW4
- SW63 pad 1: Net-(SW57-Pad1) -> ROW4
- SW64 pad 1: Net-(SW57-Pad1) -> ROW4
- SW65 pad 1: Net-(SW57-Pad1) -> ROW4
- SW7 pad 1: /key/row1 -> ROW0
- SW8 pad 1: /key/row1 -> ROW0
- SW9 pad 1: /key/row1 -> ROW0
- U1 pad 10: /PB3 -> ROW2
- U1 pad 11: /PB3 -> ROW3
- U1 pad 28: Net-(U1-Pad28) -> ROW4
- U1 pad 8: /PB0 -> ROW0
- U1 pad 9: /PB1 -> ROW1

Commit message: layout pcb
Parts:
- moved D28 214.3 mm to (274.6, 55.6), turned to 90 degrees
- moved D14 209.8 mm to (269.7, 36.6), turned to 90 degrees
- moved D27 195.2 mm to (250.7, 55.6), turned to 90 degrees
- moved D13 185.2 mm to (241.3, 36.6), turned to 90 degrees
- moved D12 170.3 mm to (222.2, 36.6), turned to 90 degrees
- moved D26 164.5 mm to (231.9, 55.6), turned to 90 degrees
- moved D25 162.4 mm to (212.6, 55.6), turned to 90 degrees
- moved D11 139.8 mm to (203.2, 36.6), turned to 90 degrees
- moved D24 139.7 mm to (193.5, 55.6), turned to 90 degrees
- moved D10 132.4 mm to (184.2, 36.6), turned to 90 degrees
- moved D22 119.6 mm to (155.4, 55.6), turned to 90 degrees
- moved D23 113.2 mm to (174.5, 55.6), turned to 90 degrees
- moved D9 105.8 mm to (165.1, 36.6), turned to 90 degrees
- moved D8 90.9 mm to (146.1, 36.6), turned to 90 degrees
- moved D21 82.3 mm to (136.4, 55.6), turned to 90 degrees
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Routing:
- net Net-(D24-Pad1): track 0.00 -> 3.18 mm
- net Net-(D23-Pad1): track 0.00 -> 3.18 mm
- net Net-(D21-Pad1): track 0.00 -> 3.18 mm
- net Net-(D14-Pad1): track 0.00 -> 3.18 mm
- net Net-(D17-Pad1): track 0.00 -> 3.18 mm
- net Net-(D20-Pad1): track 0.00 -> 3.18 mm
- net Net-(D19-Pad1): track 0.00 -> 3.18 mm
- net Net-(D18-Pad1): track 0.00 -> 3.18 mm
- net Net-(D16-Pad1): track 0.00 -> 3.18 mm
- net Net-(D27-Pad1): track 0.00 -> 3.18 mm
- net Net-(D26-Pad1): track 0.00 -> 3.18 mm
- net Net-(D25-Pad1): track 0.00 -> 3.18 mm
- net Net-(D22-Pad1): track 0.00 -> 3.18 mm
- net Net-(D15-Pad1): track 0.00 -> 3.15 mm
- net Net-(D28-Pad1): track 0.00 -> 3.15 mm
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
Commit message: layout pcb
Parts:
- moved D10 1.53 mm to (183.1, 37.7), turned to 180 degrees
- moved D21 1.32 mm to (135.4, 56.5), turned to 180 degrees
- moved D13 1.27 mm to (240.3, 37.3), turned to 180 degrees
- moved D22 1.27 mm to (154.4, 56.4), turned to 180 degrees
- moved D25 1.27 mm to (211.6, 56.4), turned to 180 degrees
- moved D28 1.27 mm to (273.6, 56.4), turned to 180 degrees
- moved D8 1.27 mm to (145.0, 37.3), turned to 180 degrees
- moved D16 1.27 mm to (40.1, 56.4), turned to 180 degrees
- moved D20 1.27 mm to (116.3, 56.4), turned to 180 degrees
- moved D5 1.27 mm to (87.9, 37.3), turned to 180 degrees
- moved D6 1.27 mm to (106.9, 37.3), turned to 180 degrees
- moved D7 1.27 mm to (126.0, 37.3), turned to 180 degrees
- moved D1 1.27 mm to (11.7, 37.3), turned to 180 degrees
- moved D15 1.27 mm to (16.5, 56.4), turned to 180 degrees
- moved D17 1.27 mm to (59.2, 56.4), turned to 180 degrees
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
Commit message: layout
Parts:
- D1, D10, D11, D12, D13, D14, D15, D16, D17, D18, D19, D2, D20, D21, D22, D23, D24, D25, D26, D27, D28, D29, D3, D30, D31, D32, D33, D34, D35, D36, D37, D38, D39, D4, D40, D41, D42, D43, D44, D45, D46, D47, D48, D49, D5, D50, D51, D52, D53, D54, D55, D56, D57, D58, D59, D6, D60, D61, D62, D63, D64, D7, D8, D9: footprint Diode_SMD:D_0805_2012Metric -> Diode_SMD:D_MiniMELF
- moved D27 1.02 mm to (248.9, 56.4)
- moved D19 1.02 mm to (96.5, 56.4)
- moved D4 1.02 mm to (67.8, 37.3)
- moved D10 0.85 mm to (182.4, 37.3)
- moved D21 0.77 mm to (134.6, 56.4)
- moved D15 0.76 mm to (15.7, 56.4)
- moved D11 0.76 mm to (201.4, 37.3)
- moved D12 0.76 mm to (220.7, 37.3)
- moved D13 0.76 mm to (239.5, 37.3)
- moved D14 0.76 mm to (268.0, 37.3)
- moved D16 0.76 mm to (39.4, 56.4)
- moved D17 0.76 mm to (58.4, 56.4)
- moved D2 0.76 mm to (30.0, 37.3)
- moved D20 0.76 mm to (115.6, 56.4)
- moved D22 0.76 mm to (153.7, 56.4)
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
Commit message: layout
Parts:
- moved D64 224.9 mm to (277.6, 113.5), turned to 180 degrees
- moved D41 212.4 mm to (265.7, 75.4), turned to 180 degrees
- moved D63 212.2 mm to (258.6, 113.5), turned to 180 degrees
- moved D54 210.5 mm to (258.6, 94.5), turned to 180 degrees
- moved D55 210.5 mm to (277.6, 94.5), turned to 180 degrees
- moved D62 190.8 mm to (239.5, 113.5), turned to 180 degrees
- moved D61 182.4 mm to (218.2, 113.5), turned to 180 degrees
- moved D53 179.5 mm to (239.5, 94.5), turned to 180 degrees
- moved D40 178.9 mm to (234.9, 75.4), turned to 180 degrees
- moved D52 166.6 mm to (220.5, 94.5), turned to 180 degrees
- moved D51 155.4 mm to (201.4, 94.5), turned to 180 degrees
- moved D38 152.8 mm to (196.8, 75.4), turned to 180 degrees
- moved D39 152.5 mm to (215.9, 75.4), turned to 180 degrees
- moved D49 129.2 mm to (163.3, 94.5), turned to 180 degrees
- moved D50 125.4 mm to (182.4, 94.5), turned to 180 degrees
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Routing:
- net Net-(D40-Pad1): track 0.00 -> 3.37 mm
- net Net-(D39-Pad1): track 0.00 -> 3.37 mm
- net Net-(D38-Pad1): track 0.00 -> 3.37 mm
- net Net-(D36-Pad1): track 0.00 -> 3.37 mm
- net Net-(D42-Pad1): track 0.00 -> 3.37 mm
- net Net-(D57-Pad1): track 0.00 -> 3.36 mm
- net Net-(D58-Pad1): track 0.00 -> 3.34 mm
- net Net-(D31-Pad1): track 0.00 -> 3.34 mm
- net Net-(D30-Pad1): track 0.00 -> 3.34 mm
- net Net-(D37-Pad1): track 0.00 -> 3.34 mm
- net Net-(D35-Pad1): track 0.00 -> 3.34 mm
- net Net-(D34-Pad1): track 0.00 -> 3.34 mm
- net Net-(D33-Pad1): track 0.00 -> 3.34 mm
- net Net-(D32-Pad1): track 0.00 -> 3.34 mm
- net Net-(D61-Pad1): track 0.00 -> 3.33 mm
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
Commit message: pcb
Parts:
- SW43: footprint Button_Switch_Keyboard:SW_Cherry_MX1A_2.00u_PCB -> Button_Switch_Keyboard:SW_Cherry_MX1A_2.25u_PCB
- SW54: footprint Button_Switch_Keyboard:SW_Cherry_MX1A_1.00u_PCB -> Button_Switch_Keyboard:SW_Cherry_MX1A_1.75u_PCB
- SW59: footprint Button_Switch_Keyboard:SW_Cherry_MX1A_1.50u_PCB -> Button_Switch_Keyboard:SW_Cherry_MX1A_1.25u_PCB
- SW62: footprint Button_Switch_Keyboard:SW_Cherry_MX1A_1.25u_PCB -> Button_Switch_Keyboard:SW_Cherry_MX1A_1.00u_PCB
- moved D51 67.5 mm to (166.7, 152.4)
- moved SW52 60.2 mm to (190.5, 152.4)
- moved SW53 14.3 mm to (214.3, 95.2)
- moved D52 14.2 mm to (206.2, 94.5)
- moved SW54 7.14 mm to (240.5, 95.2)
- moved D53 7.11 mm to (232.4, 94.5)
- moved D48 4.83 mm to (149.1, 94.5)
- moved D46 4.83 mm to (111.0, 94.5)
- moved D47 4.83 mm to (130.0, 94.5)
- moved D44 4.83 mm to (72.9, 94.5)
- moved D45 4.83 mm to (91.9, 94.5)
- moved D49 4.83 mm to (168.1, 94.5)
- moved D50 4.83 mm to (187.2, 94.5)
- moved D59 4.83 mm to (80.0, 113.5)
- moved SW48 4.76 mm to (138.1, 95.2)
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Routing:
- net Net-(D51-Pad1): track 3.31 -> 0.00 mm
